File: ENV_KB.kicad_pcb (KiCad board)
At the start: 2 copper layers, 355.7 x 160.8 mm, 177 parts

Commit message: More traces, organizing, etc.
Parts:
- removed D_7, D_8: D, CFTKB Bits:D_DO-35_SOD27_P5.08mm_Horizontal
- added D7: D, CFTKB Bits:D_DO-35_SOD27_P5.08mm_Horizontal, F.Cu at (307.6, 134.6)
- added D8: D, CFTKB Bits:D_DO-35_SOD27_P5.08mm_Horizontal, F.Cu at (326.7, 134.6)
- added G***: LOGO, EM_Logo:PersonalLogo, F.Cu at (392.9, 117.7)
- moved D27 81.7 mm to (421.6, 130.5)
- moved D43 81.7 mm to (421.6, 126.5)
- moved D60 81.7 mm to (421.6, 122.5)
- moved D74 81.7 mm to (421.6, 118.5)
- moved D82 81.7 mm to (421.6, 114.5)
- moved D9 81.7 mm to (421.6, 134.5)
- moved D10 73.2 mm to (433.1, 134.5)
- moved D28 73.2 mm to (433.1, 130.5)
- moved D44 73.2 mm to (433.1, 126.5)
- moved D61 73.2 mm to (433.1, 122.5)
- moved RPI1 62.8 mm to (352.6, 111.2)
- moved D11 61.6 mm to (442.5, 134.5)
- moved D45 61.6 mm to (442.5, 126.5)
- moved D62 61.6 mm to (442.5, 122.5)
- moved D75 61.6 mm to (442.5, 118.5)
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Routing:
- net Net-(D82-Pad2): track 125.6 -> 219.8 mm
- net Net-(D74-Pad2): track 111.2 -> 201.1 mm
- net Net-(D60-Pad2): track 89.3 -> 175.0 mm
- net Net-(D43-Pad2): track 54.2 -> 135.7 mm
- net Net-(D27-Pad2): track 40.7 -> 118.0 mm
- net Net-(D61-Pad2): track 85.4 -> 157.5 mm
- net Net-(D83-Pad2): track 118.8 -> 189.0 mm
- net Net-(D44-Pad2): track 53.4 -> 121.4 mm
- net Net-(D75-Pad2): track 105.9 -> 172.2 mm
- net Net-(D28-Pad2): track 41.6 -> 105.4 mm
- net Net-(D62-Pad2): track 86.5 -> 148.7 mm
- net Net-(D84-Pad2): track 117.5 -> 179.6 mm
- net Net-(D45-Pad2): track 52.7 -> 109.1 mm
- net Net-(D85-Pad2): track 114.7 -> 165.8 mm
- net Net-(D46-Pad2): track 87.6 -> 137.6 mm
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Other:
- board size 355.7 x 160.8 mm -> 355.8 x 176.8 mm
