File: ENV_KB.kicad_pcb (KiCad board)
At the start: 2 copper layers, 348.5 x 156.3 mm, 198 parts, among them J0 TYPE-C-31-M-12

Commit message: Front plate design adjustments to fit MCU
Parts:
- added G***: LOGO, EM_Extras:plogo, F.Cu at (454.0, 213.3)
Other:
- board text removed: "ANSI BACKSLASH"
- board text removed: "ANSI ENTER KEY"
- board text removed: "ANSI L-SHIFT"
- board text removed: "ISO Backslash"
- board text removed: "ISO ENTER"
- board text removed: "ISO L-SHIFT"
- board text removed: "ISO NUMBERSIGN"

Commit message: Adding more mount holes and some alignment adjustments
Parts:
- added H10: MountingHole, MountingHole:MountingHole_2.2mm_M2, F.Cu at (473.1, 161.8)
- added H9: MountingHole, MountingHole:MountingHole_2.2mm_M2, F.Cu at (144.6, 161.8)
- moved H5 19.3 mm to (139.9, 242.8)
- moved H4 5.52 mm to (480.2, 242.8)
- moved H7 0.65 mm to (308.6, 257.1)
- moved H2 0.22 mm to (463.6, 257.1)
Routing:
- net Net-(D64-Pad2): track 134.9 -> 135.4 mm
Other:
- board text added: "This scale is 10CM long"

Commit message: moved a bunch of traces and made the board slimmer
Parts:
- moved H4 1.90 mm to (478.3, 242.8)
- moved H5 0.55 mm to (139.3, 242.8)
- moved H0 0.18 mm to (139.2, 110.2)
Routing:
- net Net-(D77-Pad2): track 121.8 -> 209.5 mm
- net Net-(D88-Pad2): track 142.3 -> 227.5 mm
- net Net-(D49-Pad2): track 72.8 -> 156.8 mm
- net Net-(D32-Pad2): track 49.3 -> 131.3 mm
- net Net-(D87-Pad2): track 145.3 -> 197.1 mm
- net Net-(D48-Pad2): track 75.3 -> 126.4 mm
- net Net-(D31-Pad2): track 51.8 -> 100.8 mm
- net Net-(D33-Pad2): track 81.6 -> 66.2 mm
- net Net-(D50-Pad2): track 106.8 -> 91.9 mm
- net Net-(D86-Pad2): track 153.2 -> 166.6 mm
- net Net-(D47-Pad2): track 83.7 -> 95.9 mm
- net Net-(D30-Pad2): track 60.3 -> 71.4 mm
- net Net-(D64-Pad2): track 135.4 -> 124.6 mm
- net Net-(D78-Pad2): track 148.7 -> 142.4 mm
- net Net-(D16-Pad2): track 48.7 -> 43.9 mm
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Other:
- board size 348.5 x 156.3 mm -> 348.1 x 156.3 mm

Commit message: General housekeeping
Routing:
- net GND: vias 2 -> 3

Commit message: Removed un-needed via and adjusted traces for ground plane fill.
Routing:
- net GND: vias 3 -> 2

Commit message: Corrected Trace issue and added Gerber files
I added a Gerber zip, BOM and position files so you can send those off to JLCPCB if you want your own keyboard PCBs made.
Routing:
- net col0: track 347.8 -> 353.1 mm
