File: ENV_KB_temp_import_keys.sch (KiCad schematic (older format))
At the start: 218 parts, among them J1 TYPE-C-31-M-12, U1 MCP23017_SP

Commit message: Placing of the Keys and Track to the IO Expander Header for Spare Pin on IO Expander
Parts:
- removed I2CHeader1: Conn_01x04, Connector_PinSocket_2.54mm:PinSocket_1x04_P2.54mm_Vertical, symbol Connector_Generic:Conn_01x04
- removed J1: TYPE-C-31-M-12, EM_Extras:USB_C_Receptacle_HRO_TYPE-C-31-M-12, symbol Type-C-Lib:TYPE-C-31-M-12
- removed PowerLED1: Green Power Led, LED_SMD:LED_0805_2012Metric_Castellated, symbol Device:LED
- removed PowerLedResistor1: 1K Resistor, Resistor_SMD:R_0805_2012Metric, symbol Device:R_Small
- removed RESISTOR1, RESISTOR2: 5.1kohm, Resistor_SMD:R_0402_1005Metric, symbol Device:R_Small
- added P1: USB_C_Plug_USB2.0, Connector_USB:USB_C_Receptacle_HRO_TYPE-C-31-M-12, symbol Connector:USB_C_Plug_USB2.0
- D0, D1, D10, D100, D101, D102, D103, D104, D11, D12, D13, D14, D15, D16, D17, D18, D19, D2, D20, D21, D22, D23, D24, D25, D26, D27, D28, D29, D3, D30, D31, D32, D33, D34, D35, D36, D37, D38, D39, D4, D40, D41, D42, D43, D44, D45, D46, D47, D48, D49, D5, D50, D51, D52, D53, D54, D55, D56, D57, D58, D59, D6, D60, D61, D62, D63, D64, D65, D66, D67, D68, D69, D7, D70, D71, D72, D73, D74, D75, D76, D77, D78, D79, D8, D80, D81, D82, D83, D84, D85, D86, D87, D88, D89, D9, D90, D91, D92, D93, D94, D95, D96, D97, D98, D99: footprint CFTKB Bits:D_DO-35_SOD27_P5.08mm_Horizontal -> cftkb:D_DO-35_SOD27_P5.08mm_Horizontal
- K_0, K_1, K_10, K_11, K_12, K_13, K_14, K_15, K_16, K_17, K_18, K_19, K_2, K_20, K_21, K_22, K_23, K_24, K_25, K_26, K_27, K_28, K_3, K_30, K_31, K_32, K_34, K_35, K_36, K_37, K_38, K_39, K_4, K_40, K_41, K_42, K_43, K_44, K_45, K_47, K_48, K_49, K_5, K_51, K_52, K_53, K_54, K_55, K_56, K_57, K_58, K_59, K_6, K_60, K_61, K_62, K_64, K_65, K_66, K_67, K_68, K_69, K_7, K_70, K_71, K_72, K_73, K_74, K_76, K_8, K_85, K_86, K_87, K_9: footprint MX_only:MXOnly-1U-NoLED -> MX_Only:MXOnly-1U-NoLED
- K_103, K_104: footprint MX_Only:MXOnly-2U-NoLED -> MX_Only:MXOnly-1.5U-Vertical-NoLED
- K_29: footprint MX_only:MXOnly-2U-NoLED -> MX_Only:MXOnly-1U-NoLED
- K_33: footprint MX_only:MXOnly-1.5U-NoLED -> MX_Only:MXOnly-1.5U-NoLED
- K_46: footprint MX_only:MXOnly-ISO-ROTATED-ReversedStabilizers-NoLED -> MX_Only:MXOnly-ISO-ROTATED-ReversedStabilizers-NoLED
- K_50: footprint MX_only:MXOnly-1.75U-NoLED -> MX_Only:MXOnly-1.75U-NoLED
- K_63, K_77, K_78, K_79, K_81, K_82, K_83, K_84: footprint MX_only:MXOnly-1.25U-NoLED -> MX_Only:MXOnly-1.25U-NoLED
- K_75: footprint MX_only:MXOnly-2.75U-NoLED -> MX_Only:MXOnly-2.75U-NoLED
- K_80: footprint MX_only:MXOnly-6.25U-ReversedStabilizers-NoLED -> MX_Only:MXOnly-6.25U-ReversedStabilizers-NoLED
- RPI1: footprint EM_Extras:RPi_Pico_SMD_TH -> MCU_RaspberryPi_and_Boards.pretty:RPi_Pico_SMD_TH
Connections:
- net labels added: SCK, SDA, col21
- net labels removed: 3.3V, GND, I2CSCL, I2CSDA
- wire segments 471 -> 467
