File: MainPCB_RGB/ENV_KB_RGB.sch (KiCad schematic (older format))
At the start: 297 parts

Commit message: Implemented Hotswap sockets onto RGB version
Parts:
- K_0, K_1, K_10, K_11, K_12, K_13, K_14, K_15, K_16, K_17, K_18, K_19, K_2, K_20, K_21, K_22, K_23, K_24, K_25, K_26, K_27, K_28, K_3, K_30, K_31, K_32, K_34, K_35, K_36, K_37, K_38, K_39, K_4, K_40, K_41, K_42, K_43, K_44, K_45, K_47, K_48, K_49, K_5, K_51, K_52, K_53, K_54, K_55, K_56, K_57, K_58, K_59, K_6, K_60, K_61, K_62, K_65, K_66, K_67, K_68, K_69, K_7, K_70, K_71, K_72, K_73, K_74, K_75, K_77, K_8, K_86, K_87, K_88, K_9: footprint MX_Only:MXOnly-1U-NoLED -> MX_Only:MXOnly-1U-Hotswap
- K_29: footprint MX_Only:MXOnly-2U-NoLED -> MX_Only:MXOnly-2U-Hotswap
- K_33, K_46: footprint MX_Only:MXOnly-1.5U-NoLED -> MX_Only:MXOnly-1.5U-Hotswap
- K_50: footprint MX_Only:MXOnly-1.75U-NoLED -> MX_Only:MXOnly-1.75U-Hotswap
- K_63: footprint MX_only:MXOnly-ISO-ROTATED-ReversedStabilizers-NoLED -> MX_Only:MXOnly-2U-Hotswap
- K_63B1, K_64B1: footprint MX_Only:MXOnly-2.25U-NoLED -> MX_Only:MXOnly-2.25U-Hotswap
- K_64, K_78, K_79, K_80, K_82, K_83, K_84, K_85: footprint MX_Only:MXOnly-1.25U-NoLED -> MX_Only:MXOnly-1.25U-Hotswap
- K_76: footprint MX_Only:MXOnly-2.75U-NoLED -> MX_Only:MXOnly-2.75U-Hotswap
- K_81: footprint MX_Only:MXOnly-6.25U-ReversedStabilizers-NoLED -> MX_Only:MXOnly-6.25U-Hotswap-ReversedStabilizers

Commit message: Changed all mount holes to M2 and added some pads around the holes to avoid scratches being visible on pcbs
Parts:
- H0, H1, H10, H3, H4, H6, H7, H9: footprint MountingHole:MountingHole_3.2mm_M3 -> MountingHole:MountingHole_2.2mm_M2_Pad
Changed lines of the file:
@@
 EELAYER 30 0
 EELAYER END
-$Descr A0 46811 33110
+$Descr User 35433 11811
 encoding utf-8
 Sheet 1 1
@@
 F 0 "H9" H 6700 10696 50  0000 L CNN
 F 1 "MountingHole" H 6700 10605 50  0000 L CNN
-F 2 "MountingHole:MountingHole_3.2mm_M3" H 6600 10650 50  0001 C CNN
+F 2 "MountingHole:MountingHole_2.2mm_M2_Pad" H 6600 10650 50  0001 C CNN
 F 3 "~" H 6600 10650 50  0001 C CNN
 	1    6600 10650
@@
 F 0 "H10" H 6700 10896 50  0000 L CNN
 F 1 "MountingHole" H 6700 10805 50  0000 L CNN
-F 2 "MountingHole:MountingHole_3.2mm_M3" H 6600 10850 50  0001 C CNN
+F 2 "MountingHole:MountingHole_2.2mm_M2_Pad" H 6600 10850 50  0001 C CNN
 F 3 "~" H 6600 10850 50  0001 C CNN
 	1    6600 10850
@@
 F 0 "H7" H 6700 10296 50  0000 L CNN
 F 1 "MountingHole" H 6700 10205 50  0000 L CNN
-F 2 "MountingHole:MountingHole_3.2mm_M3" H 6600 10250 50  0001 C CNN
+F 2 "MountingHole:MountingHole_2.2mm_M2_Pad" H 6600 10250 50  0001 C CNN
 F 3 "~" H 6600 10250 50  0001 C CNN
 	1    6600 10250
@@
 F 0 "H6" H 6700 10096 50  0000 L CNN
 F 1 "MountingHole" H 6700 10005 50  0000 L CNN
-F 2 "MountingHole:MountingHole_3.2mm_M3" H 6600 10050 50  0001 C CNN
+F 2 "MountingHole:MountingHole_2.2mm_M2_Pad" H 6600 10050 50  0001 C CNN
 F 3 "~" H 6600 10050 50  0001 C CNN
 	1    6600 10050
@@
 F 0 "H4" H 6700 9696 50  0000 L CNN
 F 1 "MountingHole" H 6700 9605 50  0000 L CNN
-F 2 "MountingHole:MountingHole_3.2mm_M3" H 6600 9650 50  0001 C CNN
+F 2 "MountingHole:MountingHole_2.2mm_M2_Pad" H 6600 9650 50  0001 C CNN
 F 3 "~" H 6600 9650 50  0001 C CNN
 	1    6600 9650
@@
 F 0 "H1" H 6700 9096 50  0000 L CNN
 F 1 "MountingHole" H 6700 9005 50  0000 L CNN
-F 2 "MountingHole:MountingHole_3.2mm_M3" H 6600 9050 50  0001 C CNN
+F 2 "MountingHole:MountingHole_2.2mm_M2_Pad" H 6600 9050 50  0001 C CNN
 F 3 "~" H 6600 9050 50  0001 C CNN
 	1    6600 9050
@@
 F 0 "H3" H 6700 9496 50  0000 L CNN
 F 1 "MountingHole" H 6700 9405 50  0000 L CNN
-F 2 "MountingHole:MountingHole_3.2mm_M3" H 6600 9450 50  0001 C CNN
+F 2 "MountingHole:MountingHole_2.2mm_M2_Pad" H 6600 9450 50  0001 C CNN
 F 3 "~" H 6600 9450 50  0001 C CNN
 	1    6600 9450
@@
 F 0 "H0" H 6700 8896 50  0000 L CNN
 F 1 "MountingHole" H 6700 8805 50  0000 L CNN
-F 2 "MountingHole:MountingHole_3.2mm_M3" H 6600 8850 50  0001 C CNN
+F 2 "MountingHole:MountingHole_2.2mm_M2_Pad" H 6600 8850 50  0001 C CNN
 F 3 "~" H 6600 8850 50  0001 C CNN
 	1    6600 8850
