File: SwitchPlate/ENV_KB-Top.sch (KiCad schematic (older format))
At the start: 9 parts

Commit message: updated some bits namely R1 keymap
Parts:
- H0, H1, H10, H3, H4, H6, H7, H8, H9: footprint MountingHole:MountingHole_3.2mm_M3 -> mounthole:MountingHole_3.2mm_M3_modified
Changed lines of the file:
@@
 F 0 "H8" H 4600 5196 50  0000 L CNN
 F 1 "MountingHole" H 4600 5105 50  0000 L CNN
-F 2 "MountingHole:MountingHole_3.2mm_M3" H 4500 5150 50  0001 C CNN
+F 2 "mounthole:MountingHole_3.2mm_M3_modified" H 4500 5150 50  0001 C CNN
 F 3 "~" H 4500 5150 50  0001 C CNN
 	1    4500 5150
@@
 F 0 "H9" H 4600 5396 50  0000 L CNN
 F 1 "MountingHole" H 4600 5305 50  0000 L CNN
-F 2 "MountingHole:MountingHole_3.2mm_M3" H 4500 5350 50  0001 C CNN
+F 2 "mounthole:MountingHole_3.2mm_M3_modified" H 4500 5350 50  0001 C CNN
 F 3 "~" H 4500 5350 50  0001 C CNN
 	1    4500 5350
@@
 F 0 "H10" H 4600 5596 50  0000 L CNN
 F 1 "MountingHole" H 4600 5505 50  0000 L CNN
-F 2 "MountingHole:MountingHole_3.2mm_M3" H 4500 5550 50  0001 C CNN
+F 2 "mounthole:MountingHole_3.2mm_M3_modified" H 4500 5550 50  0001 C CNN
 F 3 "~" H 4500 5550 50  0001 C CNN
 	1    4500 5550
@@
 F 0 "H7" H 4600 4996 50  0000 L CNN
 F 1 "MountingHole" H 4600 4905 50  0000 L CNN
-F 2 "MountingHole:MountingHole_3.2mm_M3" H 4500 4950 50  0001 C CNN
+F 2 "mounthole:MountingHole_3.2mm_M3_modified" H 4500 4950 50  0001 C CNN
 F 3 "~" H 4500 4950 50  0001 C CNN
 	1    4500 4950
@@
 F 0 "H6" H 4600 4796 50  0000 L CNN
 F 1 "MountingHole" H 4600 4705 50  0000 L CNN
-F 2 "MountingHole:MountingHole_3.2mm_M3" H 4500 4750 50  0001 C CNN
+F 2 "mounthole:MountingHole_3.2mm_M3_modified" H 4500 4750 50  0001 C CNN
 F 3 "~" H 4500 4750 50  0001 C CNN
 	1    4500 4750
@@
 F 0 "H4" H 4600 4396 50  0000 L CNN
 F 1 "MountingHole" H 4600 4305 50  0000 L CNN
-F 2 "MountingHole:MountingHole_3.2mm_M3" H 4500 4350 50  0001 C CNN
+F 2 "mounthole:MountingHole_3.2mm_M3_modified" H 4500 4350 50  0001 C CNN
 F 3 "~" H 4500 4350 50  0001 C CNN
 	1    4500 4350
@@
 F 0 "H1" H 4600 3796 50  0000 L CNN
 F 1 "MountingHole" H 4600 3705 50  0000 L CNN
-F 2 "MountingHole:MountingHole_3.2mm_M3" H 4500 3750 50  0001 C CNN
+F 2 "mounthole:MountingHole_3.2mm_M3_modified" H 4500 3750 50  0001 C CNN
 F 3 "~" H 4500 3750 50  0001 C CNN
 	1    4500 3750
@@
 F 0 "H3" H 4600 4196 50  0000 L CNN
 F 1 "MountingHole" H 4600 4105 50  0000 L CNN
-F 2 "MountingHole:MountingHole_3.2mm_M3" H 4500 4150 50  0001 C CNN
+F 2 "mounthole:MountingHole_3.2mm_M3_modified" H 4500 4150 50  0001 C CNN
 F 3 "~" H 4500 4150 50  0001 C CNN
 	1    4500 4150
@@
 F 0 "H0" H 4600 3596 50  0000 L CNN
 F 1 "MountingHole" H 4600 3505 50  0000 L CNN
-F 2 "MountingHole:MountingHole_3.2mm_M3" H 4500 3550 50  0001 C CNN
+F 2 "mounthole:MountingHole_3.2mm_M3_modified" H 4500 3550 50  0001 C CNN
 F 3 "~" H 4500 3550 50  0001 C CNN
 	1    4500 3550

Commit message: Changed all mount holes to M2 and added some pads around the holes to avoid scratches being visible on pcbs
Parts:
- H0, H1, H10, H3, H4, H6, H7, H8, H9: footprint mounthole:MountingHole_3.2mm_M3_modified -> MountingHole:MountingHole_2.2mm_M2_Pad
Changed lines of the file:
@@
 F 0 "H8" H 4600 5196 50  0000 L CNN
 F 1 "MountingHole" H 4600 5105 50  0000 L CNN
-F 2 "mounthole:MountingHole_3.2mm_M3_modified" H 4500 5150 50  0001 C CNN
+F 2 "MountingHole:MountingHole_2.2mm_M2_Pad" H 4500 5150 50  0001 C CNN
 F 3 "~" H 4500 5150 50  0001 C CNN
 	1    4500 5150
@@
 F 0 "H9" H 4600 5396 50  0000 L CNN
 F 1 "MountingHole" H 4600 5305 50  0000 L CNN
-F 2 "mounthole:MountingHole_3.2mm_M3_modified" H 4500 5350 50  0001 C CNN
+F 2 "MountingHole:MountingHole_2.2mm_M2_Pad" H 4500 5350 50  0001 C CNN
 F 3 "~" H 4500 5350 50  0001 C CNN
 	1    4500 5350
@@
 F 0 "H10" H 4600 5596 50  0000 L CNN
 F 1 "MountingHole" H 4600 5505 50  0000 L CNN
-F 2 "mounthole:MountingHole_3.2mm_M3_modified" H 4500 5550 50  0001 C CNN
+F 2 "MountingHole:MountingHole_2.2mm_M2_Pad" H 4500 5550 50  0001 C CNN
 F 3 "~" H 4500 5550 50  0001 C CNN
 	1    4500 5550
@@
 F 0 "H7" H 4600 4996 50  0000 L CNN
 F 1 "MountingHole" H 4600 4905 50  0000 L CNN
-F 2 "mounthole:MountingHole_3.2mm_M3_modified" H 4500 4950 50  0001 C CNN
+F 2 "MountingHole:MountingHole_2.2mm_M2_Pad" H 4500 4950 50  0001 C CNN
 F 3 "~" H 4500 4950 50  0001 C CNN
 	1    4500 4950
@@
 F 0 "H6" H 4600 4796 50  0000 L CNN
 F 1 "MountingHole" H 4600 4705 50  0000 L CNN
-F 2 "mounthole:MountingHole_3.2mm_M3_modified" H 4500 4750 50  0001 C CNN
+F 2 "MountingHole:MountingHole_2.2mm_M2_Pad" H 4500 4750 50  0001 C CNN
 F 3 "~" H 4500 4750 50  0001 C CNN
 	1    4500 4750
@@
 F 0 "H4" H 4600 4396 50  0000 L CNN
 F 1 "MountingHole" H 4600 4305 50  0000 L CNN
-F 2 "mounthole:MountingHole_3.2mm_M3_modified" H 4500 4350 50  0001 C CNN
+F 2 "MountingHole:MountingHole_2.2mm_M2_Pad" H 4500 4350 50  0001 C CNN
 F 3 "~" H 4500 4350 50  0001 C CNN
 	1    4500 4350
@@
 F 0 "H1" H 4600 3796 50  0000 L CNN
 F 1 "MountingHole" H 4600 3705 50  0000 L CNN
-F 2 "mounthole:MountingHole_3.2mm_M3_modified" H 4500 3750 50  0001 C CNN
+F 2 "MountingHole:MountingHole_2.2mm_M2_Pad" H 4500 3750 50  0001 C CNN
 F 3 "~" H 4500 3750 50  0001 C CNN
 	1    4500 3750
@@
 F 0 "H3" H 4600 4196 50  0000 L CNN
 F 1 "MountingHole" H 4600 4105 50  0000 L CNN
-F 2 "mounthole:MountingHole_3.2mm_M3_modified" H 4500 4150 50  0001 C CNN
+F 2 "MountingHole:MountingHole_2.2mm_M2_Pad" H 4500 4150 50  0001 C CNN
 F 3 "~" H 4500 4150 50  0001 C CNN
 	1    4500 4150
@@
 F 0 "H0" H 4600 3596 50  0000 L CNN
 F 1 "MountingHole" H 4600 3505 50  0000 L CNN
-F 2 "mounthole:MountingHole_3.2mm_M3_modified" H 4500 3550 50  0001 C CNN
+F 2 "MountingHole:MountingHole_2.2mm_M2_Pad" H 4500 3550 50  0001 C CNN
 F 3 "~" H 4500 3550 50  0001 C CNN
 	1    4500 3550
