File: MainPCB/ENV_KB.kicad_pcb (KiCad board)
At the start: 2 copper layers, 354.6 x 156.1 mm, 197 parts

Commit message: cleanup and some small fixes as per DRC
Routing:
- net GND: track 5.70 -> 7.17 mm

Commit message: Corrected a mistake in the silkscreen, overlapping a contributor initials and footprint
Other:
- board text added: "TYVM to everyone who helped me with this project."
- board text added: "UU"
- board text removed: "Envious.Media"

Commit message: Changed all mount holes to M2 and added some pads around the holes to avoid scratches being visible on pcbs
Parts:
- H0, H1, H10, H3, H4, H6, H7, H9: footprint MountingHole:MountingHole_3.2mm_M3 -> MountingHole:MountingHole_2.2mm_M2_Pad
- PowerLedResistor0: value 1K Resistor 0402 -> 2.2K Resistor 0402
Other:
- board text removed: "TYVM to everyone who helped me with this project."
