File: AcrylicBase/Acrylic.kicad_pcb (KiCad board)
At the start: 2 copper layers, 354.6 x 156.1 mm, 8 parts

Commit message: Implemented Hotswap sockets onto RGB version
Parts:
- added G***: LOGO, EM_Logo:KBLogo, F.Cu at (357.1, 168.5)
- moved H6 0.15 mm to (212.2, 116.1)
Routing:
- net Net-(D20-Pad2): track 0.00 -> 0.79 mm
- removed copper zone on B.Cu, net GND
- removed copper zone on F.Cu, net GND
Other:
- board text added: "PLEASE CHECK ALIGNMENT OF "HRO-TYPE-C-31-M-12""

Commit message: Changed all mount holes to M2 and added some pads around the holes to avoid scratches being visible on pcbs
Parts:
- H0, H1, H10, H3, H4, H6, H7, H9: footprint mount:MountingHole_3.2mm_M3_MODIFIED -> MountingHole:MountingHole_2.2mm_M2_Pad

Commit message: updated switch plate(s) to include a slot for installing pcb mount stabs
Routing:
- net Net-(D20-Pad2): track 0.79 -> 0.00 mm
- added copper zone on B.Cu, net (none)
- added copper zone on F.Cu, net (none)
