File: MainPCB_RP2040/ENV_KB_RP2040.kicad_pcb (KiCad board)
At the start: 2 copper layers, 354.6 x 156.1 mm, 225 parts, among them J2 B3U-1000P, J5 Conn_01x03_Male, U1 AP2127K-3.3, U3 RP2040, X1 XO 32 12Mhz 3225 seiko

Commit message: Started Rework of RP2040 version (again)
Parts:
- removed the G*** at (285.0, 76.8)
- removed J5: Conn_01x03_Male, Connector_PinHeader_2.54mm:PinHeader_1x03_P2.54mm_Vertical
- removed LED3: LED 0402 YELLOW, LED_SMD:LED_0402_1005Metric
- removed PowerLED0: LED 0402, LED_SMD:LED_0402_1005Metric
- removed PowerLedResistor0: 2.2K Resistor 0402, Resistor_SMD:R_0402_1005Metric
- removed R8: 470 ohm resistor, Resistor_SMD:R_0402_1005Metric
- added C16: 18pf 0402, Capacitor_SMD:C_0402_1005Metric, F.Cu at (264.4, 83.1)
- added C18: 100nf 0201, Capacitor_SMD:C_0201_0603Metric, F.Cu at (264.6, 69.4)
- added R7: 1K 0201, Resistor_SMD:R_0201_0603Metric, F.Cu at (264.3, 81.4)
- C10, C3: value 1uf 0402 -> 1uf 0201; footprint Capacitor_SMD:C_0402_1005Metric -> Capacitor_SMD:C_0201_0603Metric
- C11, C13, C14, C15, C5, C6, C7, C8: value 100nf 0402 -> 100nf 0201; footprint Capacitor_SMD:C_0402_1005Metric -> Capacitor_SMD:C_0201_0603Metric
- C12: value 1uF 0402 -> 1uf 0201; footprint Capacitor_SMD:C_0402_1005Metric -> Capacitor_SMD:C_0201_0603Metric
- C17: value 10uf 0402 -> 100nf 0201; footprint Capacitor_SMD:C_0402_1005Metric -> Capacitor_SMD:C_0201_0603Metric
- C2: value 15pf 0402 -> 18pf 0402
- D0, D1, D10, D11, D12, D13, D14, D15, D16, D17, D18, D19, D2, D20, D21, D22, D23, D24, D25, D26, D27, D28, D29, D3, D30, D31, D32, D33, D34, D35, D36, D37, D38, D39, D4, D40, D41, D42, D43, D44, D45, D46, D47, D48, D49, D5, D50, D51, D52, D53, D54, D55, D56, D57, D58, D59, D6, D60, D61, D62, D63, D64, D65, D66, D67, D68, D69, D7, D70, D71, D72, D73, D74, D75, D76, D77, D78, D79, D8, D80, D81, D82, D83, D84, D85, D86, D87, D88, D9: value D -> 1n4148 DO-35
- Diode1: value SCHOTTKY DIODE -> 1n4002; footprint Diode_SMD:D_0603_1608Metric -> Diode_SMD:D_SOD-123
- FLASH1: footprint Package_SO:SOIC-8_5.275x5.275mm_P1.27mm -> Package_SON:SON-8-1EP_3x2mm_P0.5mm_EP1.4x1.6mm
- R1: value 1k Resistor -> 1K 0201; footprint Capacitor_SMD:C_0402_1005Metric -> Capacitor_SMD:C_0201_0603Metric
- R2: value DNF -> 10K 0402
- R4: value 27Ohms 0402 Resistor -> 27Ohms 0402 Resistor
- R5, R6: value 5.1K -> 5.1K 0402
- SW-RST0: value B3U-1000 -> SKRK; footprint Button_Switch_SMD:SW_SPST_B3U-1000P -> Button_Switch_SMD:SW_Push_SPST_NO_Alps_SKRK
- U1: value AP2127K-3.3 -> TLV75533PDBV
- X1: value XO 32 12Mhz 3225 seiko -> 3225_4P Crystal; footprint Crystal:Crystal_SMD_SeikoEpson_TSX3225-4Pin_3.2x2.5mm -> Crystal:Crystal_SMD_3225-4Pin_3.2x2.5mm
- moved C12 33.2 mm to (267.2, 63.0), turned to 90 degrees
- moved U1 31.6 mm to (269.4, 64.8), turned to 270 degrees
- moved Diode1 29.3 mm to (264.1, 63.3), turned to 0 degrees
- moved C4 28.4 mm to (270.9, 67.2), turned to 0 degrees
- moved C1 25.9 mm to (261.1, 62.8)
- moved C9 24.6 mm to (268.0, 67.2), turned to 180 degrees
- moved C7 15.0 mm to (265.1, 79.7), turned to 270 degrees
- moved J2 13.4 mm to (254.0, 68.6)
- moved R1 13.0 mm to (257.4, 68.6)
- moved C17 12.7 mm to (258.8, 75.3), turned to 180 degrees
- moved R2 12.1 mm to (257.5, 70.8), turned to 180 degrees
- moved C13 11.9 mm to (269.5, 75.3), turned to 0 degrees
- moved C10 11.4 mm to (266.8, 69.4), turned to 90 degrees
- moved FLASH1 10.0 mm to (260.7, 68.4)
- moved SW-RST0 9.22 mm to (275.1, 68.6)
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Connections:
- net Resetbtn renamed /RUN
- net USBVBUS renamed VBUS
- C10 pad 1: 3.3V -> +3V3
- C11 pad 1: 3.3V -> +3V3
- C13 pad 1: 3.3V -> +3V3
- C14 pad 1: 3.3V -> +3V3
- C15 pad 1: 3.3V -> +3V3
- C17 pad 1: 3.3V -> +3V3
- C4 pad 1: 3.3V -> +3V3
- C5 pad 1: 3.3V -> +3V3
- C8 pad 1: 3.3V -> +3V3
- C9 pad 1: 3.3V -> Net-(C9-Pad1)
- FLASH1 pad 8: 3.3V -> +3V3
- R2 pad 1: 3.3V -> +3V3
- U1 pad 4: Net-(U1-Pad4) -> Net-(C9-Pad1)
- U1 pad 5: 3.3V -> +3V3
- U3 pad 1: 3.3V -> +3V3
- U3 pad 10: 3.3V -> +3V3
- U3 pad 22: 3.3V -> +3V3
- U3 pad 33: 3.3V -> +3V3
- U3 pad 35: /GPIO23 -> row4
- U3 pad 36: /GPIO24 -> row5
- U3 pad 37: /GPIO25 -> row6
- U3 pad 38: row4 -> (no net)
- U3 pad 39: row5 -> (no net)
- U3 pad 40: row6 -> (no net)
- U3 pad 41: /GPIO29_ADC3 -> (no net)
- U3 pad 42: 3.3V -> +3V3
- U3 pad 43: 3.3V -> +3V3
- U3 pad 44: 3.3V -> +3V3
- U3 pad 48: 3.3V -> +3V3
- U3 pad 49: 3.3V -> +3V3
- X1 pad 4: 3.3V -> GND
- e1 pad 3: Net-(e1-Pad3) -> (no net)
- e1 pad 9: Net-(e1-Pad9) -> (no net)
Routing:
- net 3.3V: track 69.0 -> 0.00 mm, vias 4 -> 0
- net row0: track 401.6 -> 448.9 mm, vias 1 -> 0
- net row2: track 393.9 -> 438.1 mm, vias 1 -> 0
- net row4: track 335.6 -> 376.6 mm, vias 1 -> 0
- net row3: track 389.0 -> 429.9 mm, vias 1 -> 0
- net GND: track 55.4 -> 16.6 mm, vias 21 -> 13
- net col0: track 375.2 -> 337.6 mm, vias 1 -> 0
- net row5: track 356.2 -> 393.4 mm, vias 1 -> 0
- net col17: track 221.2 -> 184.3 mm, vias 1 -> 0
- net col16: track 202.0 -> 165.8 mm, vias 1 -> 0
- net col1: track 323.1 -> 287.2 mm, vias 1 -> 0
- net col14: track 199.9 -> 164.0 mm, vias 1 -> 0
- net col15: track 181.1 -> 146.3 mm, vias 1 -> 0
- net row6: track 371.8 -> 406.2 mm, vias 1 -> 0
- net col2: track 295.7 -> 261.6 mm, vias 1 -> 0
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- added copper zone on F.Cu, net +3V3
- removed copper zone on B.Cu, net +1V1
- removed copper zone on B.Cu, net 3.3V
- removed copper zone on F.Cu, net 3.3V
- removed copper zone on F.Cu, net VBUS
- removed copper zone on F.Cu, net VSYS
Other:
- board text removed: "CW"
- board text removed: "GP25"
- board text removed: "I am not yet sentient."
- board text removed: "PWR Present"
- board text removed: "RP2040"
- board text removed: "SWCLK"
- board text removed: "SWD"
- board text removed: "UU"
