File: MainPCB_RP2040/ENV_KB_RP2040.sch (KiCad schematic (older format))
At the start: 226 parts, among them J2 B3U-1000P, J5 Conn_01x03_Male, U1 TPS63002, U3 RP2040, X1 XO 32 12Mhz 3225 seiko

Commit message: Changed all mount holes to M2 and added some pads around the holes to avoid scratches being visible on pcbs
Parts:
- H0, H1, H10, H3, H4, H6, H7, H9: footprint MountingHole:MountingHole_3.2mm_M3 -> MountingHole:MountingHole_2.2mm_M2_Pad
Changed lines of the file:
@@
 F 0 "H9" H 6150 9796 50  0000 L CNN
 F 1 "MountingHole" H 6150 9705 50  0000 L CNN
-F 2 "MountingHole:MountingHole_3.2mm_M3" H 6050 9750 50  0001 C CNN
+F 2 "MountingHole:MountingHole_2.2mm_M2_Pad" H 6050 9750 50  0001 C CNN
 F 3 "~" H 6050 9750 50  0001 C CNN
 	1    6050 9750
@@
 F 0 "H10" H 6150 9996 50  0000 L CNN
 F 1 "MountingHole" H 6150 9905 50  0000 L CNN
-F 2 "MountingHole:MountingHole_3.2mm_M3" H 6050 9950 50  0001 C CNN
+F 2 "MountingHole:MountingHole_2.2mm_M2_Pad" H 6050 9950 50  0001 C CNN
 F 3 "~" H 6050 9950 50  0001 C CNN
 	1    6050 9950
@@
 F 0 "H7" H 6150 9596 50  0000 L CNN
 F 1 "MountingHole" H 6150 9505 50  0000 L CNN
-F 2 "MountingHole:MountingHole_3.2mm_M3" H 6050 9550 50  0001 C CNN
+F 2 "MountingHole:MountingHole_2.2mm_M2_Pad" H 6050 9550 50  0001 C CNN
 F 3 "~" H 6050 9550 50  0001 C CNN
 	1    6050 9550
@@
 F 0 "H6" H 6150 9396 50  0000 L CNN
 F 1 "MountingHole" H 6150 9305 50  0000 L CNN
-F 2 "MountingHole:MountingHole_3.2mm_M3" H 6050 9350 50  0001 C CNN
+F 2 "MountingHole:MountingHole_2.2mm_M2_Pad" H 6050 9350 50  0001 C CNN
 F 3 "~" H 6050 9350 50  0001 C CNN
 	1    6050 9350
@@
 F 0 "H4" H 6150 9196 50  0000 L CNN
 F 1 "MountingHole" H 6150 9105 50  0000 L CNN
-F 2 "MountingHole:MountingHole_3.2mm_M3" H 6050 9150 50  0001 C CNN
+F 2 "MountingHole:MountingHole_2.2mm_M2_Pad" H 6050 9150 50  0001 C CNN
 F 3 "~" H 6050 9150 50  0001 C CNN
 	1    6050 9150
@@
 F 0 "H1" H 6150 8796 50  0000 L CNN
 F 1 "MountingHole" H 6150 8705 50  0000 L CNN
-F 2 "MountingHole:MountingHole_3.2mm_M3" H 6050 8750 50  0001 C CNN
+F 2 "MountingHole:MountingHole_2.2mm_M2_Pad" H 6050 8750 50  0001 C CNN
 F 3 "~" H 6050 8750 50  0001 C CNN
 	1    6050 8750
@@
 F 0 "H3" H 6150 8996 50  0000 L CNN
 F 1 "MountingHole" H 6150 8905 50  0000 L CNN
-F 2 "MountingHole:MountingHole_3.2mm_M3" H 6050 8950 50  0001 C CNN
+F 2 "MountingHole:MountingHole_2.2mm_M2_Pad" H 6050 8950 50  0001 C CNN
 F 3 "~" H 6050 8950 50  0001 C CNN
 	1    6050 8950
@@
 F 0 "H0" H 6150 8596 50  0000 L CNN
 F 1 "MountingHole" H 6150 8505 50  0000 L CNN
-F 2 "MountingHole:MountingHole_3.2mm_M3" H 6050 8550 50  0001 C CNN
+F 2 "MountingHole:MountingHole_2.2mm_M2_Pad" H 6050 8550 50  0001 C CNN
 F 3 "~" H 6050 8550 50  0001 C CNN
 	1    6050 8550

Commit message: Mostly Completed this design but needs overall improvement
Changed lines of the file:
@@
 	0    -1   -1   0
 $EndComp
-Text GLabel 15100 5400 2    50   Input ~ 0
+Text GLabel 15000 5400 2    50   Input ~ 0
 row6
-Text GLabel 15100 5600 2    50   Input ~ 0
+Text GLabel 15000 5600 2    50   Input ~ 0
 row5
-Text GLabel 15100 6100 2    50   Input ~ 0
+Text GLabel 15000 6100 2    50   Input ~ 0
 row2
-Text GLabel 15100 5900 2    50   Input ~ 0
+Text GLabel 15000 5900 2    50   Input ~ 0
 row3
-Text GLabel 15100 5700 2    50   Input ~ 0
+Text GLabel 15000 5700 2    50   Input ~ 0
 row4
-Text GLabel 15100 6300 2    50   Input ~ 0
-col14
-Text GLabel 15100 6400 2    50   Input ~ 0
-col15
-Text GLabel 15100 6200 2    50   Input ~ 0
+Text GLabel 15000 6200 2    50   Input ~ 0
 row0
-Text GLabel 14000 5300 2    50   Input ~ 0
-col9
-Text GLabel 14000 5400 2    50   Input ~ 0
-col8
-Text GLabel 14000 5100 2    50   Input ~ 0
-col11
-Text GLabel 14000 5200 2    50   Input ~ 0
-col10
-Text GLabel 14000 4900 2    50   Input ~ 0
-col12
-Text GLabel 14000 4800 2    50   Input ~ 0
-col13
-Text GLabel 14000 5900 2    50   Input ~ 0
-col4
-Text GLabel 14000 5800 2    50   Input ~ 0
-col5
-Text GLabel 14000 5700 2    50   Input ~ 0
-col6
-Text GLabel 14000 5600 2    50   Input ~ 0
-col7
-Text GLabel 14000 6100 2    50   Input ~ 0
-col3
-Text GLabel 14000 6400 2    50   Input ~ 0
-col0
-Text GLabel 14000 6300 2    50   Input ~ 0
-col1
-Text GLabel 14000 6200 2    50   Input ~ 0
-col2
-Text GLabel 15100 6700 2    50   Input ~ 0
-col17
-Text GLabel 15100 6600 2    50   Input ~ 0
-col16
-Text GLabel 15000 4800 2    50   Input ~ 0
+Text GLabel 14900 4800 2    50   Input ~ 0
 USBVBUS
-Text GLabel 14000 6500 2    50   Input ~ 0
+Text GLabel 13950 6500 2    50   Input ~ 0
 GND
-Text GLabel 14000 6000 2    50   Input ~ 0
+Text GLabel 13950 6000 2    50   Input ~ 0
 GND
-Text GLabel 14000 5500 2    50   Input ~ 0
+Text GLabel 13950 5500 2    50   Input ~ 0
 GND
-Text GLabel 14000 5000 2    50   Input ~ 0
+Text GLabel 13950 5000 2    50   Input ~ 0
 GND
-Text GLabel 15100 6500 2    50   Input ~ 0
+Text GLabel 15000 6500 2    50   Input ~ 0
 GND
-Text GLabel 15100 6000 2    50   Input ~ 0
+Text GLabel 15000 6000 2    50   Input ~ 0
 GND
-Text GLabel 15100 5000 2    50   Input ~ 0
+Text GLabel 15000 5000 2    50   Input ~ 0
 GND
 Wire Wire Line
@@
 	-1   0    0    1
 $EndComp
-Text GLabel 13900 6700 2    50   Input ~ 0
+Text GLabel 13850 6700 2    50   Input ~ 0
 I2CSDA
-Text GLabel 13900 6600 2    50   Input ~ 0
+Text GLabel 13850 6600 2    50   Input ~ 0
 I2CSCL
-Text GLabel 15000 5200 2    50   Input ~ 0
+Text GLabel 14900 5200 2    50   Input ~ 0
 3.3V
 Text GLabel 14100 8350 2    50   Input ~ 0
@@
 Text GLabel 14100 8550 2    50   Input ~ 0
 3.3V
-Text GLabel 15000 5800 2    50   Input ~ 0
+Text GLabel 14900 5800 2    50   Input ~ 0
 Resetbtn
 Text GLabel 11900 8650 0    50   Input ~ 0
@@
 Wire Wire Line
 	14400 6300 15000 6300
+Text GLabel 15000 6400 2    50   Input ~ 0
+col16
+Text GLabel 15000 6300 2    50   Input ~ 0
+col17
+Text GLabel 15000 6600 2    50   Input ~ 0
+col15
+Text GLabel 15000 6700 2    50   Input ~ 0
+col14
+Text GLabel 13950 4800 2    50   Input ~ 0
+col13
+Text GLabel 13950 4900 2    50   Input ~ 0
+col12
+Text GLabel 13950 5200 2    50   Input ~ 0
+col10
+Text GLabel 13950 5100 2    50   Input ~ 0
+col11
+Text GLabel 13950 5400 2    50   Input ~ 0
+col8
+Text GLabel 13950 5300 2    50   Input ~ 0
+col9
+Text GLabel 13950 5600 2    50   Input ~ 0
+col7
+Text GLabel 13950 5700 2    50   Input ~ 0
+col6
+Text GLabel 13950 5800 2    50   Input ~ 0
+col5
+Text GLabel 13950 5900 2    50   Input ~ 0
+col4
+Text GLabel 13950 6200 2    50   Input ~ 0
+col2
+Text GLabel 13950 6300 2    50   Input ~ 0
+col1
+Text GLabel 13950 6400 2    50   Input ~ 0
+col0
+Text GLabel 13950 6100 2    50   Input ~ 0
+col3
 $EndSCHEMATC

Commit message: replaced buck boost with a LDO (AP2127K-3.3)
Parts:
- removed L1: Inductor 2.2uh, Inductor_SMD:L_0805_2012Metric, symbol Device:L_Small
- removed R7: 100ohm, Resistor_SMD:R_0402_1005Metric, symbol Device:R
- removed U1: TPS63002, Package_SON:Texas_DRC0010J_ThermalVias, symbol Regulator_Switching:TPS63002
- added U1: AP2127K-3.3, Package_TO_SOT_SMD:SOT-23-5, symbol Regulator_Linear:AP2127K-3.3
- C12: value 0.1uf 0402 -> 1uF 0402
Connections:
- net 3V3_EN is gone; now on net VBUS: C12.1
- net +3V3: now also U1.5 (VOUT)
- net GND: now also U1.2 (GND)
- net VBUS: now also U1.1 (VIN), U1.3 (EN)
Changed lines of the file:
@@
 Wire Wire Line
 	2450 1900 2450 1850
-Text GLabel 14900 5100 0    50   Input ~ 0
-3V3_EN
 $Comp
 L W25Q256JVEIQ_TR:W25Q256JVEIQ_TR FLASH1
@@
 Text Notes 900  850  0    50   ~ 0
 2x 5.1K Resistors on the CC pins will = 5V@1.5A\nthis is the recomended default config for type-c
-Text GLabel 2900 2250 0    50   Input ~ 0
-3V3_EN
-$Comp
-L Device:R R7
-U 1 1 608CFAF0
-P 2900 2100
-F 0 "R7" H 2750 2150 50  0000 L CNN
-F 1 "100ohm" V 2900 2050 30  0000 L CNN
-F 2 "Resistor_SMD:R_0402_1005Metric" V 2830 2100 50  0001 C CNN
-F 3 "" H 2900 2100 50  0001 C CNN
-	1    2900 2100
-	1    0    0    -1
-$EndComp
-Wire Wire Line
-	2900 1950 2900 1850
 $Comp
 L power:GND #PWR0110
 U 1 1 60C62E0C
-P 4000 2650
-F 0 "#PWR0110" H 4000 2400 50  0001 C CNN
-F 1 "GND" H 4005 2477 50  0000 C CNN
-F 2 "" H 4000 2650 50  0001 C CNN
-F 3 "" H 4000 2650 50  0001 C CNN
-	1    4000 2650
+P 4100 2250
+F 0 "#PWR0110" H 4100 2000 50  0001 C CNN
+F 1 "GND" H 4105 2077 50  0000 C CNN
+F 2 "" H 4100 2250 50  0001 C CNN
+F 3 "" H 4100 2250 50  0001 C CNN
+	1    4100 2250
 	1    0    0    -1
 $EndComp
 Wire Wire Line
 	2200 1750 2200 1850
-$Comp
-L power:GND #PWR0111
-U 1 1 60C8A405
-P 3100 2450
-F 0 "#PWR0111" H 3100 2200 50  0001 C CNN
-F 1 "GND" H 3105 2277 50  0000 C CNN
-F 2 "" H 3100 2450 50  0001 C CNN
-F 3 "" H 3100 2450 50  0001 C CNN
-	1    3100 2450
-	1    0    0    -1
-$EndComp
-$Comp
-L Device:L_Small L1
-U 1 1 60C9C176
-P 4100 1300
-F 0 "L1" V 4400 1300 50  0000 C CNN
-F 1 "Inductor 2.2uh" V 4250 1300 50  0000 C CNN
-F 2 "Inductor_SMD:L_0805_2012Metric" H 4100 1300 50  0001 C CNN
-F 3 "~" H 4100 1300 50  0001 C CNN
-	1    4100 1300
-	0    -1   -1   0
-$EndComp
 $Comp
 L Simulation_SPICE:DIODE Diode1
@@
 	2550 1850 2450 1850
 Wire Wire Line
-	2850 1850 2900 1850
-Connection ~ 2900 1850
-Wire Wire Line
-	2900 1850 3100 1850
-Wire Wire Line
 	3100 1850 3100 1700
 Connection ~ 3100 1850
@@
 Text Label 2300 1850 0    50   ~ 0
 VBUS
-$Comp
-L Regulator_Switching:TPS63002 U1
-U 1 1 60D7C270
-P 4100 2050
-F 0 "U1" H 4100 2717 50  0000 C CNN
-F 1 "TPS63002" H 4100 2626 50  0000 C CNN
-F 2 "Package_SON:Texas_DRC0010J_ThermalVias" H 4950 1500 50  0001 C CNN
-F 3 "http://www.ti.com/lit/ds/symlink/tps63000.pdf" H 3800 2600 50  0001 C CNN
-	1    4100 2050
-	1    0    0    -1
-$EndComp
 Wire Wire Line
 	5200 1750 5200 1850
-Wire Wire Line
-	3700 1650 3700 1300
-Wire Wire Line
-	3700 1300 4000 1300
-Wire Wire Line
-	4500 1650 4500 1300
-Wire Wire Line
-	4500 1300 4200 1300
-Wire Wire Line
-	3100 1850 3700 1850
-Wire Wire Line
-	3300 2250 3300 2050
-Wire Wire Line
-	3300 1950 3700 1950
-Wire Wire Line
-	2900 2250 3100 2250
-Wire Wire Line
-	3700 2050 3300 2050
-Connection ~ 3300 2050
-Wire Wire Line
-	3300 2050 3300 1950
-Wire Wire Line
-	3700 2250 3300 2250
-Connection ~ 3300 2250
-$Comp
-L Device:C_Small C12
-U 1 1 60E73823
-P 3100 2350
-F 0 "C12" H 3192 2396 50  0000 L CNN
-F 1 "0.1uf 0402" H 3192 2305 50  0000 L CNN
-F 2 "Capacitor_SMD:C_0402_1005Metric" H 3100 2350 50  0001 C CNN
-F 3 "~" H 3100 2350 50  0001 C CNN
-	1    3100 2350
-	1    0    0    -1
-$EndComp
-Connection ~ 3100 2250
-Wire Wire Line
-	3100 2250 3300 2250
 $Comp
 L Device:C C9
@@
 	5200 1850 4900 1850
 Connection ~ 5200 1850
-Wire Wire Line
-	4500 1850 4650 1850
 Connection ~ 4900 1850
-Wire Wire Line
-	4500 2050 4650 2050
-Wire Wire Line
-	4650 2050 4650 1850
-Connection ~ 4650 1850
-Wire Wire Line
-	4650 1850 4900 1850
-$Comp
-L power:GND #PWR05
-U 1 1 60EAD68C
-P 4100 2650
-F 0 "#PWR05" H 4100 2400 50  0001 C CNN
-F 1 "GND" H 4105 2477 50  0000 C CNN
-F 2 "" H 4100 2650 50  0001 C CNN
-F 3 "" H 4100 2650 50  0001 C CNN
-	1    4100 2650
-	1    0    0    -1
-$EndComp
 Wire Wire Line
 	13350 4800 13950 4800
@@
 Text GLabel 13950 6100 2    50   Input ~ 0
 col3
+$Comp
+L Regulator_Linear:AP2127K-3.3 U1
+U 1 1 6107E6AC
+P 4100 1950
+F 0 "U1" H 4100 2292 50  0000 C CNN
+F 1 "AP2127K-3.3" H 4100 2201 50  0000 C CNN
+F 2 "Package_TO_SOT_SMD:SOT-23-5" H 4100 2275 50  0001 C CNN
+F 3 "https://www.diodes.com/assets/Datasheets/AP2127.pdf" H 4100 2050 50  0001 C CNN
+	1    4100 1950
+	1    0    0    -1
+$EndComp
+Wire Wire Line
+	4400 1850 4900 1850
+Wire Wire Line
+	2850 1850 3100 1850
+$Comp
+L Device:C_Small C12
+U 1 1 6119F94E
+P 3700 2100
+F 0 "C12" H 3650 2150 20  0000 L CNN
+F 1 "1uF 0402" H 3650 2100 20  0000 L CNN
+F 2 "Capacitor_SMD:C_0402_1005Metric" H 3700 2100 50  0001 C CNN
+F 3 "~" H 3700 2100 50  0001 C CNN
+	1    3700 2100
+	1    0    0    -1
+$EndComp
+$Comp
+L power:GND #PWR0111
+U 1 1 611A0432
+P 3700 2200
+F 0 "#PWR0111" H 3700 1950 50  0001 C CNN
+F 1 "GND" H 3705 2027 50  0000 C CNN
+F 2 "" H 3700 2200 50  0001 C CNN
+F 3 "" H 3700 2200 50  0001 C CNN
+	1    3700 2200
+	1    0    0    -1
+$EndComp
+Wire Wire Line
+	3100 1850 3700 1850
+Wire Wire Line
+	3700 2000 3700 1950
+Wire Wire Line
+	3700 1950 3800 1950
+Wire Wire Line
+	3700 1950 3700 1850
+Connection ~ 3700 1950
+Connection ~ 3700 1850
+Wire Wire Line
+	3700 1850 3800 1850
 $EndSCHEMATC

Commit message: corrected all DRC Errors, all vias on pads as well as separated vbus and vsys in the schematic properly.
Parts:
- added TP1, TP2, TP3: TestPoint, TestPoint:TestPoint_Pad_D1.5mm, symbol Connector:TestPoint
Connections:
- net GPIO23: now also TP3.1
- net GPIO24: now also TP2.1
- net GPIO29_ADC3: now also TP1.1
- net VBUS: no longer C12.1, Diode1.2 (K), U1.1 (VIN), U1.3 (EN)
- new net VSYS: C12.1, Diode1.2 (K), U1.1 (VIN), U1.3 (EN)
Changed lines of the file:
@@
 	2550 1850 2450 1850
-Wire Wire Line
-	3100 1850 3100 1700
-Connection ~ 3100 1850
-$Comp
-L VSYS:VSYS #PWR0112
-U 1 1 60D018CC
-P 3100 1700
-F 0 "#PWR0112" H 3100 1550 50  0001 C CNN
-F 1 "VSYS" H 3115 1873 50  0000 C CNN
-F 2 "" H 3100 1700 50  0001 C CNN
-F 3 "" H 3100 1700 50  0001 C CNN
-	1    3100 1700
-	1    0    0    -1
-$EndComp
 Wire Wire Line
 	14900 4900 14850 4900
@@
 Wire Wire Line
 	14600 5200 14900 5200
-Text Label 3250 1850 0    50   ~ 0
-VSYS
 Text Label 2300 1850 0    50   ~ 0
 VBUS
@@
 Text GLabel 13950 6100 2    50   Input ~ 0
 col3
+Wire Wire Line
+	4400 1850 4900 1850
+$Comp
+L Device:C_Small C12
+U 1 1 6119F94E
+P 3700 2100
+F 0 "C12" H 3650 2150 20  0000 L CNN
+F 1 "1uF 0402" H 3650 2100 20  0000 L CNN
+F 2 "Capacitor_SMD:C_0402_1005Metric" H 3700 2100 50  0001 C CNN
+F 3 "~" H 3700 2100 50  0001 C CNN
+	1    3700 2100
+	1    0    0    -1
+$EndComp
+$Comp
+L power:GND #PWR0111
+U 1 1 611A0432
+P 3700 2200
+F 0 "#PWR0111" H 3700 1950 50  0001 C CNN
+F 1 "GND" H 3705 2027 50  0000 C CNN
+F 2 "" H 3700 2200 50  0001 C CNN
+F 3 "" H 3700 2200 50  0001 C CNN
+	1    3700 2200
+	1    0    0    -1
+$EndComp
+Wire Wire Line
+	3700 2000 3700 1950
+Wire Wire Line
+	3700 1950 3800 1950
+Wire Wire Line
+	3700 1950 3700 1850
+Connection ~ 3700 1950
+Wire Wire Line
+	3700 1850 3800 1850
 $Comp
 L Regulator_Linear:AP2127K-3.3 U1
@@
 	1    0    0    -1
 $EndComp
-Wire Wire Line
-	4400 1850 4900 1850
-Wire Wire Line
-	2850 1850 3100 1850
-$Comp
-L Device:C_Small C12
-U 1 1 6119F94E
-P 3700 2100
-F 0 "C12" H 3650 2150 20  0000 L CNN
-F 1 "1uF 0402" H 3650 2100 20  0000 L CNN
-F 2 "Capacitor_SMD:C_0402_1005Metric" H 3700 2100 50  0001 C CNN
-F 3 "~" H 3700 2100 50  0001 C CNN
-	1    3700 2100
-	1    0    0    -1
-$EndComp
-$Comp
-L power:GND #PWR0111
-U 1 1 611A0432
-P 3700 2200
-F 0 "#PWR0111" H 3700 1950 50  0001 C CNN
-F 1 "GND" H 3705 2027 50  0000 C CNN
-F 2 "" H 3700 2200 50  0001 C CNN
-F 3 "" H 3700 2200 50  0001 C CNN
-	1    3700 2200
-	1    0    0    -1
-$EndComp
-Wire Wire Line
-	3100 1850 3700 1850
-Wire Wire Line
-	3700 2000 3700 1950
-Wire Wire Line
-	3700 1950 3800 1950
-Wire Wire Line
-	3700 1950 3700 1850
-Connection ~ 3700 1950
+$Comp
+L Connector:TestPoint TP1
+U 1 1 612D2ECF
+P 15850 4300
+F 0 "TP1" H 15908 4418 50  0000 L CNN
+F 1 "TestPoint" H 15908 4327 50  0000 L CNN
+F 2 "TestPoint:TestPoint_Pad_D1.5mm" H 16050 4300 50  0001 C CNN
+F 3 "~" H 16050 4300 50  0001 C CNN
+	1    15850 4300
+	1    0    0    -1
+$EndComp
+$Comp
+L Connector:TestPoint TP2
+U 1 1 612D4ABD
+P 16300 4300
+F 0 "TP2" H 16358 4418 50  0000 L CNN
+F 1 "TestPoint" H 16358 4327 50  0000 L CNN
+F 2 "TestPoint:TestPoint_Pad_D1.5mm" H 16500 4300 50  0001 C CNN
+F 3 "~" H 16500 4300 50  0001 C CNN
+	1    16300 4300
+	1    0    0    -1
+$EndComp
+$Comp
+L Connector:TestPoint TP3
+U 1 1 612D5578
+P 16800 4300
+F 0 "TP3" H 16858 4418 50  0000 L CNN
+F 1 "TestPoint" H 16858 4327 50  0000 L CNN
+F 2 "TestPoint:TestPoint_Pad_D1.5mm" H 17000 4300 50  0001 C CNN
+F 3 "~" H 17000 4300 50  0001 C CNN
+	1    16800 4300
+	1    0    0    -1
+$EndComp
+Wire Wire Line
+	15850 4300 15850 4900
+Text Label 15850 4900 1    50   ~ 0
+GPIO29_ADC3
+Wire Wire Line
+	16800 4300 16800 4900
+Wire Wire Line
+	16300 4300 16300 4900
+Text Label 16800 4900 1    50   ~ 0
+GPIO23
+Text Label 16300 4900 1    50   ~ 0
+GPIO24
+Text GLabel 3350 1850 0    50   Input ~ 0
+VSYS
+Text GLabel 2850 1850 2    50   Input ~ 0
+VSYS
+Wire Wire Line
+	3350 1850 3700 1850
 Connection ~ 3700 1850
-Wire Wire Line
-	3700 1850 3800 1850
 $EndSCHEMATC

Commit message: Started Rework of RP2040 version (again)
Parts:
- removed LED3: LED 0402 YELLOW, LED_SMD:LED_0402_1005Metric, symbol Device:LED
- removed PowerLED0: LED 0402, LED_SMD:LED_0402_1005Metric, symbol Device:LED
- removed PowerLedResistor0: 2.2K Resistor 0402, Resistor_SMD:R_0402_1005Metric, symbol Device:R_Small
- removed R8: 470 ohm resistor, Resistor_SMD:R_0402_1005Metric, symbol Device:R
- removed TP1, TP2, TP3: TestPoint, TestPoint:TestPoint_Pad_D1.5mm, symbol Connector:TestPoint
- added C16: 18pf 0402, Capacitor_SMD:C_0402_1005Metric, symbol Device:C
- added C18: 100nf 0201, Capacitor_SMD:C_0201_0603Metric, symbol Device:C
- added R7: 1K 0201, Resistor_SMD:R_0201_0603Metric, symbol Device:R_Small
- C10, C3: value 1uf 0402 -> 1uf 0201; footprint Capacitor_SMD:C_0402_1005Metric -> Capacitor_SMD:C_0201_0603Metric
- C11, C13, C14, C15, C5, C6, C7, C8: value 100nf 0402 -> 100nf 0201; footprint Capacitor_SMD:C_0402_1005Metric -> Capacitor_SMD:C_0201_0603Metric
- C12: value 1uF 0402 -> 1uf 0201; footprint Capacitor_SMD:C_0402_1005Metric -> Capacitor_SMD:C_0201_0603Metric
- C17: value 10uf 0402 -> 100nf 0201; footprint Capacitor_SMD:C_0402_1005Metric -> Capacitor_SMD:C_0201_0603Metric
- C2: value 15pf 0402 -> 18pf 0402
- D0, D1, D10, D11, D12, D13, D14, D15, D16, D17, D18, D19, D2, D20, D21, D22, D23, D24, D25, D26, D27, D28, D29, D3, D30, D31, D32, D33, D34, D35, D36, D37, D38, D39, D4, D40, D41, D42, D43, D44, D45, D46, D47, D48, D49, D5, D50, D51, D52, D53, D54, D55, D56, D57, D58, D59, D6, D60, D61, D62, D63, D64, D65, D66, D67, D68, D69, D7, D70, D71, D72, D73, D74, D75, D76, D77, D78, D79, D8, D80, D81, D82, D83, D84, D85, D86, D87, D88, D9: value D -> 1n4148 DO-35
- Diode1: value SCHOTTKY DIODE -> 1n4002; footprint Diode_SMD:D_0603_1608Metric -> Diode_SMD:D_SOD-123
- FLASH1: footprint Package_SO:SOIC-8_5.275x5.275mm_P1.27mm -> Package_SON:SON-8-1EP_3x2mm_P0.5mm_EP1.4x1.6mm
- J2: value B3U-1000P -> SKRK; footprint Button_Switch_SMD:SW_SPST_B3U-1000P -> Button_Switch_SMD:SW_Push_SPST_NO_Alps_SKRK
- R1: value 1k Resistor -> 1K 0201; footprint Capacitor_SMD:C_0402_1005Metric -> Capacitor_SMD:C_0201_0603Metric
- R2: value DNF -> 10K 0402
- R4: value 27Ohms 0402 Resistor -> 27Ohms 0402 Resistor
- R5, R6: value 5.1K -> 5.1K 0402
- SW-RST0: value B3U-1000 -> SKRK; footprint Button_Switch_SMD:SW_SPST_B3U-1000P -> Button_Switch_SMD:SW_Push_SPST_NO_Alps_SKRK
- U1: value AP2127K-3.3 -> TLV75533PDBV; symbol Regulator_Linear:AP2127K-3.3 -> Regulator_Linear:LDK130-08_SOT23_SOT353
- X1: value XO 32 12Mhz 3225 seiko -> 3225_4P Crystal; footprint Crystal:Crystal_SMD_SeikoEpson_TSX3225-4Pin_3.2x2.5mm -> Crystal:Crystal_SMD_3225-4Pin_3.2x2.5mm; symbol Oscillator:XO32 -> Device:Crystal_GND24
Connections:
- net GPIO23 is gone; now on net row4: U3.35 (GPIO23)
- net GPIO24 is gone; now on net row5: U3.36 (GPIO24)
- net GPIO25 is gone; now on net row6: U3.37 (GPIO25)
- net +3V3: now also C18.1; no longer C9.1, I2CHeader0.2 (Pin_2), X1.4 (V+)
- net GND: now also FLASH1.9 (EXP), X1.4, C16.1, C18.2
- net XOUT: now also R7.1
- net row4: no longer U3.38 (GPIO26_ADC0)
- net row5: no longer U3.39 (GPIO27_ADC1)
- net row6: no longer U3.40 (GPIO28_ADC2)
- net at X1.1: now also C16.2, R7.2
- net at U1.4 (BP): now also C9.1
- net Resetbtn renamed RUN
- new net 3.3V: I2CHeader0.2 (Pin_2)
- new net GPIO26_ADC0: U3.38 (GPIO26_ADC0)
- new net GPIO27_ADC1: U3.39 (GPIO27_ADC1)
- new net GPIO28_ADC2: U3.40 (GPIO28_ADC2)
- no-connect marks 0 -> 2
Other:
- note added: "If I recall right, RP2040 supports 1 to 16MHz"
- note removed: "Dont bother trying to use a crystal\nas it massively complicates this clock source setup"
- note removed: "Intentionally left floating"
- note removed: "Pin1 on XO Oscillator also left floating so the chip is enabled\n(this is specified in their datasheet)"
- note removed: "Use a 12mhz Seiko Oscilator, 3225-4Pin"
- moved on the sheet: C2, C9, I2CHeader0, J5, SW-RST0
