File: MainPCB_RP2040/ENV_KB_RP2040.kicad_sch (KiCad schematic)
At the start: 224 parts, among them J2 SKRK, J5 Conn_01x03_Male, U1 TLV75533PDBV, U3 RP2040, X1 3225_4P Crystal

Commit message: Added EEPROM to RP2040 version
Parts:
- removed e1: TYPE-C-31-M-12, HRO-TYPE-C31-M-12:HRO-TYPE-C-31-M-12, symbol Type-C:HRO-TYPE-C-31-M-12
- added R8, R9: 10K 0402 Resistor, Capacitor_SMD:C_0402_1005Metric, symbol Device:R
- added U2: 24LC64, Package_SO:SOIC-8-1EP_3.9x4.9mm_P1.27mm_EP2.29x3mm, symbol Memory_EEPROM:24LC64
- added e1: TYPE_C_31_M-14, josh-connectors:USB_C_TYPE-C-31-M-14, symbol josh-connector:USB_C_U262-161N-4BVC11
Connections:
- net +3V3: now also R8.1, R9.1, U2.8 (VCC)
- net GND: now also U2.1 (A0), U2.2 (A1), U2.3 (A2), U2.4 (GND), U2.7 (WP), e1.A1 (GND), e1.A12 (GND), e1.B1 (GND), e1.B12 (GND), e1.S1 (SHIELD)
- net I2CSCL: now also R9.2, U2.6 (SCL)
- net I2CSDA: now also R8.2, U2.5 (SDA)
- net USB_D+: now also e1.A6 (D+), e1.B6 (D+)
- net USB_D-: now also e1.A7 (D-), e1.B7 (D-)
- net VBUS: now also e1.A4 (VBUS), e1.A9 (VBUS), e1.B4 (VBUS), e1.B9 (VBUS)
- net at R6.2: now also e1.A5 (CC1)
- net at R5.2: now also e1.B5 (CC2)
Other:
- note added: "EEPROM"
- note added: "EEPROM for Dynamic config storage"
- note added: "KoreanHROParts HRO_TYPE-C-31-M-14"
- note removed: "KoreanHROParts USB_C_Receptacle_HRO_TYPE-C-31-M-12"
- moved on the sheet: R5, R6

Commit message: Tidied up some stuff and updated the logo.
Parts:
- J2, SW-RST0: value SKRK -> EVQPUJ; footprint Button_Switch_SMD:SW_Push_SPST_NO_Alps_SKRK -> Button_Switch_SMD:Panasonic_EVQPUJ_EVQPUA
Changed lines of the file:
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@@
     (in_bom yes) (on_board yes)
     (property "Reference" "J2" (id 0) (at 33.02 124.46 0))
-    (property "Value" "SKRK" (id 1) (at 34.29 130.81 0))
-    (property "Footprint" "Button_Switch_SMD:SW_Push_SPST_NO_Alps_SKRK" (id 2) (at 34.29 128.27 0)
+    (property "Value" "EVQPUJ" (id 1) (at 34.29 130.81 0))
+    (property "Footprint" "Button_Switch_SMD:Panasonic_EVQPUJ_EVQPUA" (id 2) (at 34.29 128.27 0)
       (effects (font (size 1.27 1.27)) hide)
     )
@@
     (in_bom yes) (on_board yes)
     (property "Reference" "SW-RST0" (id 0) (at 148.59 170.18 0))
-    (property "Value" "SKRK" (id 1) (at 149.86 165.1 0))
-    (property "Footprint" "Button_Switch_SMD:SW_Push_SPST_NO_Alps_SKRK" (id 2) (at 154.94 167.64 0)
+    (property "Value" "EVQPUJ" (id 1) (at 149.86 165.1 0))
+    (property "Footprint" "Button_Switch_SMD:Panasonic_EVQPUJ_EVQPUA" (id 2) (at 154.94 167.64 0)
       (effects (font (size 1.27 1.27)) (justify left bottom) hide)
     )
@@
   (symbol (lib_id "power:VBUS") (at 39.37 31.75 270) (unit 1)
     (in_bom yes) (on_board yes)
-    (property "Reference" "#PWR?" (id 0) (at 35.56 31.75 0)
+    (property "Reference" "#PWR0113" (id 0) (at 35.56 31.75 0)
       (effects (font (size 1.27 1.27)) hide)
     )
@@
     )
     (path "/0f9de786-9b05-494c-90c3-759356db0d8c"
-      (reference "#PWR?") (unit 1) (value "VBUS") (footprint "")
+      (reference "#PWR0113") (unit 1) (value "VBUS") (footprint "")
     )
     (path "/00000000-0000-0000-0000-00005f09255d"
@@
     )
     (path "/00000000-0000-0000-0000-00005f30f0ba"
-      (reference "J2") (unit 1) (value "SKRK") (footprint "Button_Switch_SMD:SW_Push_SPST_NO_Alps_SKRK")
+      (reference "J2") (unit 1) (value "EVQPUJ") (footprint "Button_Switch_SMD:Panasonic_EVQPUJ_EVQPUA")
     )
     (path "/00000000-0000-0000-0000-000060ce2dd4"
@@
     )
     (path "/00000000-0000-0000-0000-0000605fbfa6"
-      (reference "SW-RST0") (unit 1) (value "SKRK") (footprint "Button_Switch_SMD:SW_Push_SPST_NO_Alps_SKRK")
+      (reference "SW-RST0") (unit 1) (value "EVQPUJ") (footprint "Button_Switch_SMD:Panasonic_EVQPUJ_EVQPUA")
     )
     (path "/00000000-0000-0000-0000-00006107e6ac"
