File: SwitchPlatePCB/ENV_KB_SWITCHPLATE.kicad_pcb (KiCad board)
At the start: 2 copper layers, 347 x 156.3 mm, 30 parts

Commit message: lots more work towards making this available
Parts:
- removed kibuzzard-628AE768: G***, kibuzzard-628AE768
- removed kibuzzard-628AE7EF: G***, kibuzzard-628AE7EF
- removed kibuzzard-628AE7FB: G***, kibuzzard-628AE7FB
- removed kibuzzard-628AE805: G***, kibuzzard-628AE805
- removed kibuzzard-628AE80F: G***, kibuzzard-628AE80F
- removed kibuzzard-628AE82F: G***, kibuzzard-628AE82F
- removed kibuzzard-628AE860: G***, kibuzzard-628AE860
- removed kibuzzard-628AE868: G***, kibuzzard-628AE868
- removed kibuzzard-628AE874: G***, kibuzzard-628AE874
- removed kibuzzard-628AE882: G***, kibuzzard-628AE882
- removed kibuzzard-628AE8A6: G***, kibuzzard-628AE8A6
- removed kibuzzard-628AE933: G***, kibuzzard-628AE933
- removed kibuzzard-628AE966: G***, kibuzzard-628AE966
- removed kibuzzard-628AEA91: G***, kibuzzard-628AEA91
Routing:
- added copper zone on B.Cu, net (none)
- added copper zone on F.Cu, net (none)
Other:
- board size 347 x 156.3 mm -> 350.6 x 127.8 mm
- board text removed: "5.1K"
- board text removed: "<Stepped NotStepped>"
- board text removed: "https://github.com/Envious-Data/Env-KB"
